Commit message: Fix the urdf.

File: urdf/mogi_bot.urdf.xacro (robot description, xacro)
@@ -176,5 +176,5 @@
   </link>
   <!-- STEP 4 - 云台偏航关节 (Yaw) -->
-  <joint name="gimbal_yaw_joint" type="revolute">
+  <joint name="gimbal_yaw_joint" type="fixed">
     <origin xyz="0 0 0.04" rpy="0 0 0" />
     <parent link="gimbal_base"/>
